Commit message: pre-release - 0.0.1

File: source/sensor_parameter/edgar.urdf (robot description, URDF)
Before this commit: robot EDGAR, 34 links, 33 joints
Links:
- link rear_axle_center_ground: geometry visual mesh filename=file:///absolute/path/to/the/3d_model/low_res/edgar.fbx scale=1 1 1

Commit message: Costum EDGAR Model

File: source/sensor_parameter/edgar.urdf (robot description, URDF)
Before this commit: robot EDGAR, 34 links, 33 joints
Links:
- link rear_axle_center_ground: geometry visual mesh filename=file:///absolute/path/to/the/3d_model/high_res/EDGAR_T7.fbx scale=0.01 0.01 0.01

Commit message: update urdf

File: source/sensor_parameter/edgar.urdf (robot description, URDF)
Before this commit: robot EDGAR, 34 links, 33 joints
Links:
- removed link camera_lr_front_left
- removed link camera_lr_front_right
- removed link camera_sr_front_center
- removed link camera_sr_front_left
- removed link camera_sr_front_right
- removed link camera_sr_rear_center
- removed link camera_sr_rear_left
- removed link camera_sr_rear_right
- removed link framos_front_left
- removed link framos_front_right
- removed link gnss_left
- removed link gnss_right
- removed link imu
- removed link lidar_innovusion_front
- removed link lidar_innovusion_rear
- removed link lidar_ouster_left
- removed link lidar_ouster_right
- removed link microphone_front_left
- removed link microphone_front_right
- removed link microphone_rear_left
- removed link microphone_rear_right
- removed link mimo_center
- removed link mimo_left
- removed link mimo_right
- removed link rack_rear_center
- removed link radar_front_center
- removed link radar_front_left
- removed link radar_front_right
- removed link radar_rear_center
- removed link radar_rear_left
- removed link radar_rear_right
- removed link rear_axle_center
- removed link rear_axle_center_ground
- added link antenna_novatel_left
- added link antenna_novatel_right
- added link antenna_panorama_center
- added link antenna_panorama_left
- added link antenna_panorama_right
- added link axle_edgar_rearcenter
- added link axle_edgar_rearcenterground; visual mesh filename=file:///absolute/path/to/the/3d_model/high_res/EDGAR_T7.fbx scale=0.01 0.01 0.01
- added link camera_basler_frontcenter
- added link camera_basler_frontcenterleft
- added link camera_basler_frontcenterright
- added link camera_basler_frontleft
- added link camera_basler_frontright
- added link camera_basler_rearcenter
- added link camera_basler_rearleft
- added link camera_basler_rearright
- added link camera_framos_frontleft
- added link camera_framos_frontright
- added link gnss_novatel_center
- added link imu_novatel_center
- added link imu_ouster_frontleft
- added link imu_ouster_frontright
- added link lidar_aeva_frontcenter
- added link lidar_innovusion_frontcenter
- added link lidar_innovusion_rearcenter
- added link lidar_ouster_frontleft
- added link lidar_ouster_frontright
- added link microphone_infineon_frontleft
- added link microphone_infineon_frontright
- added link microphone_infineon_rearleft
- added link microphone_infineon_rearright
- added link rack_edgar_rearcenter
- added link radar_continental_frontcenter
- added link radar_continental_frontleft
- added link radar_continental_frontright
- added link radar_continental_rearcenter
- added link radar_continental_rearleft
- added link radar_continental_rearright
Joints:
- removed joint camera_lr_front_left_joint
- removed joint camera_lr_front_right_joint
- removed joint camera_sr_front_center_joint
- removed joint camera_sr_front_left_joint
- removed joint camera_sr_front_right_joint
- removed joint camera_sr_rear_center_joint
- removed joint camera_sr_rear_left_joint
- removed joint camera_sr_rear_right_joint
- removed joint framos_front_left_joint
- removed joint framos_front_right_joint
- removed joint gnss_left_joint
- removed joint gnss_right_joint
- removed joint imu_joint
- removed joint lidar_innovusion_front_joint
- removed joint lidar_innovusion_rear_joint
- removed joint lidar_ouster_left_joint
- removed joint lidar_ouster_right_joint
- removed joint microphone_front_left_joint
- removed joint microphone_front_right_joint
- removed joint microphone_rear_left_joint
- removed joint microphone_rear_right_joint
- removed joint mimo_center_joint
- removed joint mimo_left_joint
- removed joint mimo_right_joint
- removed joint rack_rear_center_joint
- removed joint radar_front_center_joint
- removed joint radar_front_left_joint
- removed joint radar_front_right_joint
- removed joint radar_rear_center_joint
- removed joint radar_rear_left_joint
- removed joint radar_rear_right_joint
- removed joint rear_axle_center_ground_joint
- removed joint rear_axle_center_joint
- added joint antenna_novatel_left_joint: type fixed, parent axle_edgar_rearcenter, child antenna_novatel_left, origin xyz=1.475 0.545 1.714
- added joint antenna_novatel_right_joint: type fixed, parent axle_edgar_rearcenter, child antenna_novatel_right, origin xyz=1.475 -0.545 1.714
- added joint antenna_panorama_center_joint: type fixed, parent axle_edgar_rearcenter, child antenna_panorama_center, origin xyz=0.851 0.0 1.729 rpy=0.0 0.0 0.0
- added joint antenna_panorama_left_joint: type fixed, parent axle_edgar_rearcenter, child antenna_panorama_left, origin xyz=0.23 0.547 1.737 rpy=0.0 0.0 0.0
- added joint antenna_panorama_right_joint: type fixed, parent axle_edgar_rearcenter, child antenna_panorama_right, origin xyz=0.231 -0.548 1.737 rpy=0.0 0.0 0.0
- added joint axle_edgar_rearcenter_joint: type fixed, parent axle_edgar_rearcenterground, child axle_edgar_rearcenter, origin xyz=0.0 0.0 0.338
- added joint axle_edgar_rearcenterground_joint: type fixed, parent base_link, child axle_edgar_rearcenterground, origin xyz=0.0 0.0 0.0
- added joint camera_basler_frontcenter_joint: type fixed, parent lidar_innovusion_frontcenter, child camera_basler_frontcenter, origin xyz=0.17217 0.00830 0.10242 rpy=-0.01306798 -0.01235135 1.56602337
- added joint camera_basler_frontcenterleft_joint: type fixed, parent axle_edgar_rearcenter, child camera_basler_frontcenterleft, origin xyz=2.163 0.385 1.705 rpy=0.0 0.0 0.0
- added joint camera_basler_frontcenterright_joint: type fixed, parent axle_edgar_rearcenter, child camera_basler_frontcenterright, origin xyz=2.163 -0.385 1.705 rpy=0.0 0.0 0.0
- added joint camera_basler_frontleft_joint: type fixed, parent lidar_ouster_frontleft, child camera_basler_frontleft, origin xyz=-0.04426 0.03683 0.11894 rpy=-1.49130077 0.2840286 -0.75821117
- added joint camera_basler_frontright_joint: type fixed, parent lidar_ouster_frontright, child camera_basler_frontright, origin xyz=0.01477 0.02652 0.12120 rpy=-1.50206631 -0.32925375 -2.45009512
- added joint camera_basler_rearcenter_joint: type fixed, parent lidar_innovusion_rearcenter, child camera_basler_rearcenter, origin xyz=0.08173 -0.08121 0.27614 rpy=0.08378889 0.00332415 1.55765627
- added joint camera_basler_rearleft_joint: type fixed, parent lidar_innovusion_rearcenter, child camera_basler_rearleft, origin xyz=-0.02216 0.85016 -0.03938 rpy=0.24728924 1.05107428 1.93298793
- added joint camera_basler_rearright_joint: type fixed, parent lidar_innovusion_rearcenter, child camera_basler_rearright, origin xyz=-0.01137 -0.65154 -0.00656 rpy=-0.09417622 -0.93148048 1.40893048
- added joint camera_framos_frontleft_joint: type fixed, parent axle_edgar_rearcenter, child camera_framos_frontleft, origin xyz=2.203 0.195 1.705 rpy=0.0 0.0 0.0
- added joint camera_framos_frontright_joint: type fixed, parent axle_edgar_rearcenter, child camera_framos_frontright, origin xyz=2.203 -0.195 1.705 rpy=0.0 0.0 0.0
- added joint gnss_novatel_center_joint: type fixed, parent axle_edgar_rearcenter, child gnss_novatel_center, origin xyz=0.321 -0.007 0.208 rpy=0.0 0.0 1.5708
- added joint imu_novatel_center_joint: type fixed, parent axle_edgar_rearcenter, child imu_novatel_center, origin xyz=0.321 -0.007 0.208 rpy=0.0 0.0 0.0
- added joint imu_ouster_frontleft_joint: type fixed, parent lidar_ouster_frontleft, child imu_ouster_frontleft, origin xyz=-0.006 0.012 -0.029 rpy=0.0 0.0 3.142
- added joint imu_ouster_frontright_joint: type fixed, parent lidar_ouster_frontright, child imu_ouster_frontright, origin xyz=-0.006 0.012 -0.029 rpy=0.0 0.0 3.142
- added joint lidar_aeva_frontcenter_joint: type fixed, parent axle_edgar_rearcenter, child lidar_aeva_frontcenter, origin xyz=2.259 0.302735673 1.760425312 rpy=0.0000291 0.19 -0.035
- added joint lidar_innovusion_frontcenter_joint: type fixed, parent axle_edgar_rearcenter, child lidar_innovusion_frontcenter, origin xyz=2.259 0.0 1.600 rpy=3.14159265 -1.369065 0.0
- added joint lidar_innovusion_rearcenter_joint: type fixed, parent axle_edgar_rearcenter, child lidar_innovusion_rearcenter, origin xyz=-0.3987347 0.002735673 1.760425312 rpy=0.0000291 -1.7552732 0
- added joint lidar_ouster_frontleft_joint: type fixed, parent axle_edgar_rearcenter, child lidar_ouster_frontleft, origin xyz=2.312053 0.581505 1.610277 rpy=-0.3461248 0.0165291 -0.0162606
- added joint lidar_ouster_frontright_joint: type fixed, parent axle_edgar_rearcenter, child lidar_ouster_frontright, origin xyz=2.311906 -0.664888 1.612698 rpy=0.3551248 0.0165291 0.0061281
- added joint microphone_infineon_frontleft_joint: type fixed, parent axle_edgar_rearcenter, child microphone_infineon_frontleft, origin xyz=3.819 0.821 0.173 rpy=0.0 0.0 0.785398
- added joint microphone_infineon_frontright_joint: type fixed, parent axle_edgar_rearcenter, child microphone_infineon_frontright, origin xyz=3.817 -0.822 0.173 rpy=0.0 0.0 -0.785398
- added joint microphone_infineon_rearleft_joint: type fixed, parent axle_edgar_rearcenter, child microphone_infineon_rearleft, origin xyz=-0.701 0.875 0.37 rpy=0.0 0.0 2.32129
- added joint microphone_infineon_rearright_joint: type fixed, parent axle_edgar_rearcenter, child microphone_infineon_rearright, origin xyz=-0.7 -0.875 0.37 rpy=0.0 0.0 -2.32129
- added joint rack_edgar_rearcenter_joint: type fixed, parent axle_edgar_rearcenterground, child rack_edgar_rearcenter, origin xyz=-0.502 0.0 1.97
- added joint radar_continental_frontcenter_joint: type fixed, parent axle_edgar_rearcenter, child radar_continental_frontcenter, origin xyz=4.060 -0.220 0.043 rpy=0.0 0.0698132 0.0
- added joint radar_continental_frontleft_joint: type fixed, parent axle_edgar_rearcenter, child radar_continental_frontleft, origin xyz=3.964 0.655 0.170 rpy=0.0 0.0 0.383972
- added joint radar_continental_frontright_joint: type fixed, parent axle_edgar_rearcenter, child radar_continental_frontright, origin xyz=3.965 -0.645 0.170 rpy=0.0 0.0174533 -0.383972
- added joint radar_continental_rearcenter_joint: type fixed, parent axle_edgar_rearcenter, child radar_continental_rearcenter, origin xyz=-0.920 -0.008 0.083 rpy=0.0 0.0174533 0.0
- added joint radar_continental_rearleft_joint: type fixed, parent axle_edgar_rearcenter, child radar_continental_rearleft, origin xyz=-0.844 0.716 0.085 rpy=0.0 0.0174533 2.79253
- added joint radar_continental_rearright_joint: type fixed, parent axle_edgar_rearcenter, child radar_continental_rearright, origin xyz=-0.842 -0.715 0.085 rpy=0.0 0.0523599 -2.79253
